File: PCB/pcb.kicad_pcb (KiCad board)
At the start: 2 copper layers, 78 x 78 mm, 10 parts, among them J1 Reed, J2 Button, J3 LED, J4 Servo, M3 MountingHole_3.2mm_M3, U1 NodeMCU1.0(ESP-12E), U2 ACS712xLCTR-30A

Commit message: updated PCB design
Parts:
- moved M3 0.92 mm to (48.2, 126.6)
Routing:
- net Net-(J4-Pin_2): track 60.7 -> 65.8 mm
- net Net-(U1-VIN): track 22.3 -> 26.0 mm
Changed lines of the file:
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@@
   )
   (footprint "MountingHole:MountingHole_3.2mm_M3" (layer "F.Cu")
-    (at 48.6664 125.8316)
+    (at 48.1838 126.619)
     (descr "Mounting Hole 3.2mm, no annular, M3")
     (tags "mounting hole 3.2mm no annular m3")
@@
   (segment (start 66.9586 81.0514) (end 67.5386 81.0514) (width 0.25) (layer "F.Cu") (net 6))
   (segment (start 67.5386 81.0514) (end 78.994 81.0514) (width 0.25) (layer "F.Cu") (net 6))
-  (segment (start 67.5386 77.2414) (end 62.5886 77.2414) (width 0.25) (layer "F.Cu") (net 19))
-  (segment (start 62.5886 77.2414) (end 62.5886 78.5114) (width 0.25) (layer "F.Cu") (net 19))
-  (segment (start 62.211849 78.5114) (end 54.44 86.283249) (width 0.25) (layer "F.Cu") (net 19))
-  (segment (start 62.5886 78.5114) (end 62.211849 78.5114) (width 0.25) (layer "F.Cu") (net 19))
-  (segment (start 54.44 86.283249) (end 54.44 91.03) (width 0.25) (layer "F.Cu") (net 19))
+  (segment (start 54.44 82.6692) (end 54.44 91.03) (width 0.25) (layer "F.Cu") (net 19))
+  (segment (start 64.516 77.2414) (end 64.516 77.851) (width 0.25) (layer "F.Cu") (net 19))
+  (segment (start 63.8556 78.5114) (end 62.5886 78.5114) (width 0.25) (layer "F.Cu") (net 19))
+  (segment (start 67.5386 77.2414) (end 64.516 77.2414) (width 0.25) (layer "F.Cu") (net 19))
+  (segment (start 64.516 77.2414) (end 62.5886 77.2414) (width 0.25) (layer "F.Cu") (net 19))
+  (segment (start 58.5978 78.5114) (end 54.44 82.6692) (width 0.25) (layer "F.Cu") (net 19))
+  (segment (start 64.516 77.851) (end 63.8556 78.5114) (width 0.25) (layer "F.Cu") (net 19))
+  (segment (start 62.5886 78.5114) (end 58.5978 78.5114) (width 0.25) (layer "F.Cu") (net 19))
   (segment (start 84.92 128.308) (end 84.92 118.97) (width 0.25) (layer "F.Cu") (net 21))
   (segment (start 82.1182 131.1098) (end 84.92 128.308) (width 0.25) (layer "F.Cu") (net 21))
   (segment (start 93.868134 131.1098) (end 87.46 124.701666) (width 0.25) (layer "F.Cu") (net 30))
   (segment (start 87.46 124.701666) (end 87.46 118.97) (width 0.25) (layer "F.Cu") (net 30))
+  (segment (start 65.2272 79.9846) (end 65.2272 80.8228) (width 0.25) (layer "F.Cu") (net 31))
   (segment (start 56.896 86.744) (end 56.896 87.3252) (width 0.25) (layer "F.Cu") (net 31))
+  (segment (start 64.9986 81.0514) (end 62.5886 81.0514) (width 0.25) (layer "F.Cu") (net 31))
   (segment (start 62.5886 81.0514) (end 56.896 86.744) (width 0.25) (layer "F.Cu") (net 31))
-  (segment (start 62.5886 79.7814) (end 62.5886 81.0514) (width 0.25) (layer "F.Cu") (net 31))
+  (segment (start 65.2272 80.8228) (end 64.9986 81.0514) (width 0.25) (layer "F.Cu") (net 31))
+  (segment (start 65.024 79.7814) (end 65.2272 79.9846) (width 0.25) (layer "F.Cu") (net 31))
+  (segment (start 62.5886 79.7814) (end 65.024 79.7814) (width 0.25) (layer "F.Cu") (net 31))
   (via (at 56.896 87.3252) (size 0.8) (drill 0.4) (layers "F.Cu" "B.Cu") (net 31))
   (segment (start 50.7238 121.965266) (end 58.618334 129.8598) (width 0.25) (layer "B.Cu") (net 31))
