File: PCB/v5/smartlock_v5.kicad_pcb (KiCad board)
At the start: 2 copper layers, 69.8 x 25.2 mm, 37 parts, among them J1 USB-C, J2 battery, J3 motor, SW1 button, U1 ESP32-C6-MINI-1-N4, U2 DRV8833PW, U3 MCP73831-2, U4 RT9080-33, U5 DRV5032 (hub), U6 DRV5032 (thumb-turn)

Commit message: v5: battery and USB-powered versions, polished case, exact AliExpress links
Two versions from the same mechanism, PCB and firmware source:
- CAD: layout(door, power); the USB case has no pouch and is 3.5 mm
  shorter (59.5 vs 63.0 mm on a rosette door). case_* and light_pipe_*
  STLs per version, everything else shared. checks.py runs fit, motion,
  assembly and printability for both: 51/51 pass.
- PCB: R13 (0 ohm, VBUS -> VBAT) for the USB version; per-version BOMs
  (bom_battery.csv without R13, bom_usb.csv without charger, PROG
  resistor and battery connector). Re-placed and re-routed: KiCad DRC
  0 errors, 0 unconnected.
- Firmware: SMARTLOCK_USB_POWERED (Kconfig) + sdkconfig.defaults.usb:
  Thread FTD router, no ICD/PM, Matter power source "wired". Both builds
  pass (battery 1.55 MB, USB 1.59 MB).

Polish: V-reveals at base/case and case/cap, chamfered top edge, debossed
padlock on the cap, rounded flush flexure button with a finger dimple,
rounded USB-C opening sized for a plug moulding (the old 12 x 5.2 mm cut
was too small for a plug to seat). All downward chamfers steeper than 45
deg. Fixed: chamfer_cut severed the base's bayonet spigot (caught by the
lock check); largest() now fails if a real piece breaks off. Renders use
refined meshes (no shading streaks); new two-version render.

docs/v5-parts.md: a specific AliExpress listing and the exact variant to
pick for every bought part, per version; PCB via JLCPCB.

Co-Authored-By: Claude Opus 5.5 <noreply@anthropic.com>
Parts:
- added R13: 0R, R_0805_2012Metric, F.Cu at (77.9, 115.8)
Routing:
- net GND: track 151.4 -> 162.5 mm, vias 99 -> 102
- net HALL_HUB: track 24.3 -> 31.4 mm, vias 1 -> 5
- net MOTOR_IN1: track 23.7 -> 28.5 mm
- net ISENSE: track 48.3 -> 43.9 mm, vias 4 -> 6
- net VCP: track 17.2 -> 14.0 mm, vias 4 -> 2
- net VBAT: track 104.3 -> 101.2 mm, vias 15 -> 11
- net CHG_STAT: track 49.2 -> 52.2 mm, vias 6 -> 5
- net 3V3: track 92.8 -> 95.6 mm, vias 20 -> 15
- net VBUS: track 15.3 -> 18.0 mm
- net LED_A: track 1.71 -> 2.79 mm, vias 2 -> 0
- net EN: track 11.5 -> 10.5 mm
- net VBAT_SENSE: track 16.3 -> 15.3 mm, vias 3 -> 4
- net MOTOR_FAULT: track 36.7 -> 37.7 mm
- net MOT_A: track 12.0 -> 13.0 mm
- net MOTOR_SLEEP: track 23.1 -> 22.3 mm
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